Commit message: Update assemblyURDF_sim_v3.urdf

File: assemblyURDF_sim_v3/urdf/assemblyURDF_sim_v3.urdf (robot description, URDF)
Before this commit: robot assemblyURDF_sim_v3, 13 links, 11 joints
Joints:
- removed joint servo_4_joints
- added joint leg_1_joint: type continuous, parent servo_1_link, child leg_1_link, origin xyz=0.015 -0.013 -0.00280397218834483 rpy=0 0 0.625000267634323, axis 0 0 -1
- added joint servo_4_joint: type continuous, parent base_link, child servo_4_link, origin xyz=0.0492951218109149 0.0284532934482133 0.0239999999999998 rpy=1.2521204794546 0 3.14159265358979, axis -1 0 0
